File: hakkit_badusb.kicad_sch (KiCad schematic)
At the start: 19 parts, among them J2 Micro_SD_Card, J3 USB_A, SW1 SW_Push, U1 RP2040, U3 LT1962-3.3, U4 W25Q16JVSS, Y2 Crystal 12MHz

Commit message: final pcb must order
Parts:
- C1, C2: LCSC C1589 -> (none)
- C3: LCSC C503219 -> (none)
- C4: LCSC C14664 -> (none)
- C5, C6: LCSC C1644 -> (none)
- D2: LCSC C2846931 -> (none)
- J2: LCSC C164170 -> (none)
- J3: LCSC C386752 -> (none)
- R1, R5: LCSC C22789 -> (none)
- R2, R4: LCSC C12030 -> (none)
- R3: LCSC C12038 -> (none)
- SW1: LCSC C72443 -> (none)
- U1: LCSC C2040 -> (none)
- U3: LCSC C107774 -> (none)
- U4: LCSC C82317 -> (none)
- Y2: LCSC C70565 -> (none)
Changed lines of the file:
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@@
 			)
 		)
-		(property "LCSC" "C1644"
-			(at 72.39 125.73 0)
-			(effects
-				(font
-					(size 1.27 1.27)
-				)
-				(hide yes)
-			)
-		)
 		(pin "1"
 		)
@@
 			)
 		)
-		(property "LCSC" "C1589"
-			(at 331.47 35.5599 0)
-			(effects
-				(font
-					(size 1.27 1.27)
-				)
-				(hide yes)
-			)
-		)
 		(pin "1"
 		)
@@
 			)
 		)
-		(property "LCSC" "C72443"
-			(at 81.788 95.504 0)
-			(effects
-				(font
-					(size 1.27 1.27)
-				)
-				(hide yes)
-			)
-		)
 		(pin "2"
 		)
@@
 			)
 		)
-		(property "LCSC" "C2040"
-			(at 130.4133 151.13 0)
-			(effects
-				(font
-					(size 1.27 1.27)
-				)
-				(hide yes)
-			)
-		)
 		(pin "2"
 		)
@@
 			)
 		)
-		(property "LCSC" "C22789"
-			(at 97.79 96.266 0)
-			(effects
-				(font
-					(size 1.27 1.27)
-				)
-				(hide yes)
-			)
-		)
 		(pin "1"
 		)
@@
 			)
 		)
-		(property "LCSC" "C386752"
-			(at 229.87 22.86 0)
-			(effects
-				(font
-					(size 1.27 1.27)
-				)
-				(hide yes)
-			)
-		)
 		(pin "SH"
 		)
@@
 			)
 		)
-		(property "LCSC" "C503219"
-			(at 341.63 32.5881 0)
-			(effects
-				(font
-					(size 1.27 1.27)
-				)
-				(hide yes)
-			)
-		)
 		(pin "2"
 		)
@@
 			)
 		)
-		(property "LCSC" "C12038"
-			(at 231.14 50.038 0)
-			(effects
-				(font
-					(size 1.27 1.27)
-				)
-				(hide yes)
-			)
-		)
 		(pin "1"
 		)
@@
 			)
 		)
-		(property "LCSC" "C22789"
-			(at 97.79 87.376 0)
-			(effects
-				(font
-					(size 1.27 1.27)
-				)
-				(hide yes)
-			)
-		)
 		(pin "1"
 		)
@@
 			)
 		)
-		(property "LCSC" "C164170"
-			(at 260.985 96.52 0)
-			(effects
-				(font
-					(size 1.27 1.27)
-				)
-				(hide yes)
-			)
-		)
 		(pin "1"
 		)
@@
 			)
 		)
-		(property "LCSC" "C82317"
-			(at 44.45 107.9499 0)
-			(effects
-				(font
-					(size 1.27 1.27)
-				)
-				(hide yes)
-			)
-		)
 		(pin "2"
 		)
@@
 			)
 		)
-		(property "LCSC" "C1644"
-			(at 72.136 136.144 0)
-			(effects
-				(font
-					(size 1.27 1.27)
-				)
-				(hide yes)
-			)
-		)
 		(pin "1"
 		)
@@
 			)
 		)
-		(property "LCSC" "C107774"
-			(at 312.42 22.86 0)
-			(effects
-				(font
-					(size 1.27 1.27)
-				)
-				(hide yes)
-			)
-		)
 		(pin "4"
 		)
@@
 			)
 		)
-		(property "LCSC" "C1589"
-			(at 232.41 65.532 0)
-			(effects
-				(font
-					(size 1.27 1.27)
-				)
-				(hide yes)
-			)
-		)
 		(pin "1"
 		)
@@
 			)
 		)
-		(property "LCSC" "C12030"
-			(at 72.39 95.2499 0)
-			(effects
-				(font
-					(size 1.27 1.27)
-				)
-				(hide yes)
-			)
-		)
 		(pin "2"
 		)
@@
 			)
 		)
-		(property "LCSC" "C12030"
-			(at 231.14 103.886 0)
-			(effects
-				(font
-					(size 1.27 1.27)
-				)
-				(hide yes)
-			)
-		)
 		(pin "1"
 		)
@@
 			)
 		)
-		(property "LCSC" "C14664"
-			(at 296.672 39.37 0)
-			(effects
-				(font
-					(size 1.27 1.27)
-				)
-				(hide yes)
-			)
-		)
 		(pin "2"
 		)
@@
 			)
 		)
-		(property "LCSC" "C70565"
-			(at 86.614 129.032 0)
-			(effects
-				(font
-					(size 1.27 1.27)
-				)
-				(hide yes)
-			)
-		)
 		(pin "1"
 		)
@@
 			)
 		)
-		(property "LCSC" "C2846931"
-			(at 173.99 79.9398 0)
-			(effects
-				(font
-					(size 1.27 1.27)
-				)
-				(hide yes)
-			)
-		)

Commit message: must redo tf-01a
Parts:
- removed J2: Micro_SD_Card, Connector_Card:microSD_HC_Molex_47219-2001, symbol Connector:Micro_SD_Card
- removed R4: 10kR, Resistor_SMD:R_0603_1608Metric, symbol Device:R
- added MICRO_SD1: TF-01A, TF-01A:TF-01A, symbol TF-01A:TF-01A
- added R6: 10kR, Resistor_SMD:R_0603_1608Metric, symbol Device:R
Connections:
- net +3V3: now also MICRO_SD1.4 (VDD), R6.1
- net GND: now also MICRO_SD1.6 (VSS), MICRO_SD1.MP1 (SHIELD), MICRO_SD1.MP2 (SHIELD), MICRO_SD1.MP3 (SHIELD), MICRO_SD1.MP4 (SHIELD)
- net SD_CS: now also MICRO_SD1.2 (CD/DAT3), R6.2
- net SD_MISO: now also MICRO_SD1.7 (DAT0)
- net SD_MOSI: now also MICRO_SD1.3 (CMD)
- net SD_SCK: now also MICRO_SD1.5 (CLK)
- no-connect marks 30 -> 31
